File: intellivision t-card replic/intellivision t-card glue.kicad_sch (KiCad schematic)
At the start: 20 parts, among them SW4 SW_DIP_x08, U15 74LS51, U16 74LS00, U17 74LS85

Commit message: partial layout
Parts:
- removed C7: 100nF, Capacitor_THT:C_Disc_D3.8mm_W2.6mm_P2.50mm, symbol Device:C
Connections:
- net +5V: no longer SW4.10, SW4.11, SW4.12, SW4.13, SW4.14, SW4.15, SW4.9, U16.1, U16.2
- net GND: now also SW4.10, SW4.11, SW4.12, SW4.13, SW4.14, SW4.15, SW4.16, SW4.9, U16.1, U16.2
- no-connect marks 4 -> 3
Changed lines of the file:
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@@
   (junction (at 170.18 29.845) (diameter 0) (color 0 0 0 0)
   )
-  (junction (at 196.85 144.145) (diameter 0) (color 0 0 0 0)
-  )
   (junction (at 206.375 29.845) (diameter 0) (color 0 0 0 0)
   )
+  (junction (at 165.1 29.845) (diameter 0) (color 0 0 0 0)
+  )
   (junction (at 212.725 160.655) (diameter 0) (color 0 0 0 0)
   )
@@
   (junction (at 102.235 92.075) (diameter 0) (color 0 0 0 0)
   )
-  (junction (at 196.85 151.765) (diameter 0) (color 0 0 0 0)
-  )
   (junction (at 123.825 85.725) (diameter 0) (color 0 0 0 0)
   )
   (junction (at 172.72 29.845) (diameter 0) (color 0 0 0 0)
   )
-  (junction (at 199.39 29.845) (diameter 0) (color 0 0 0 0)
-  )
   (junction (at 180.34 29.845) (diameter 0) (color 0 0 0 0)
   )
@@
   (junction (at 100.965 64.135) (diameter 0) (color 0 0 0 0)
   )
-  (junction (at 182.88 29.845) (diameter 0) (color 0 0 0 0)
+  (junction (at 224.155 29.845) (diameter 0) (color 0 0 0 0)
   )
   (junction (at 213.36 29.845) (diameter 0) (color 0 0 0 0)
@@
   (junction (at 177.8 29.845) (diameter 0) (color 0 0 0 0)
   )
+  (junction (at 210.82 117.475) (diameter 0) (color 0 0 0 0)
+  )
   (junction (at 170.18 51.435) (diameter 0) (color 0 0 0 0)
   )
-  (junction (at 210.82 112.395) (diameter 0) (color 0 0 0 0)
-  )
   (junction (at 182.88 60.96) (diameter 0) (color 0 0 0 0)
   )
+  (junction (at 167.64 29.845) (diameter 0) (color 0 0 0 0)
+  )
   (junction (at 100.965 55.88) (diameter 0) (color 0 0 0 0)
   )
@@
   (junction (at 212.725 135.255) (diameter 0) (color 0 0 0 0)
   )
-  (no_connect (at 165.1 29.845))
   (no_connect (at 127 98.425))
   (no_connect (at 127 100.965))
@@
     (stroke (width 0) (type default) (color 0 0 0 0))
   )
-  (wire (pts (xy 196.85 151.765) (xy 184.15 151.765))
-    (stroke (width 0) (type default) (color 0 0 0 0))
-  )
   (wire (pts (xy 199.39 34.29) (xy 199.39 29.845))
     (stroke (width 0) (type default) (color 0 0 0 0))
@@
     (stroke (width 0) (type default) (color 0 0 0 0))
   )
-  (wire (pts (xy 210.82 109.855) (xy 210.82 112.395))
-    (stroke (width 0) (type default) (color 0 0 0 0))
-  )
   (wire (pts (xy 177.8 45.085) (xy 177.8 57.15))
     (stroke (width 0) (type default) (color 0 0 0 0))
   )
+  (wire (pts (xy 156.845 29.845) (xy 156.845 35.56))
+    (stroke (width 0) (type default) (color 0 0 0 0))
+  )
+  (wire (pts (xy 224.155 29.845) (xy 227.33 29.845))
+    (stroke (width 0) (type default) (color 0 0 0 0))
+  )
   (wire (pts (xy 165.1 45.085) (xy 165.1 47.625))
     (stroke (width 0) (type default) (color 0 0 0 0))
@@
     (stroke (width 0) (type default) (color 0 0 0 0))
   )
+  (wire (pts (xy 167.64 29.845) (xy 165.1 29.845))
+    (stroke (width 0) (type default) (color 0 0 0 0))
+  )
   (wire (pts (xy 210.82 112.395) (xy 210.82 117.475))
     (stroke (width 0) (type default) (color 0 0 0 0))
@@
     (stroke (width 0) (type default) (color 0 0 0 0))
   )
+  (wire (pts (xy 165.1 29.845) (xy 156.845 29.845))
+    (stroke (width 0) (type default) (color 0 0 0 0))
+  )
   (wire (pts (xy 102.235 64.135) (xy 102.235 76.835))
     (stroke (width 0) (type default) (color 0 0 0 0))
@@
     (stroke (width 0) (type default) (color 0 0 0 0))
   )
-  (wire (pts (xy 220.345 29.845) (xy 227.33 29.845))
+  (wire (pts (xy 220.345 29.845) (xy 224.155 29.845))
     (stroke (width 0) (type default) (color 0 0 0 0))
   )
@@
     (stroke (width 0) (type default) (color 0 0 0 0))
   )
-  (wire (pts (xy 182.88 29.845) (xy 199.39 29.845))
-    (stroke (width 0) (type default) (color 0 0 0 0))
-  )
   (wire (pts (xy 63.5 104.775) (xy 76.835 104.775))
     (stroke (width 0) (type default) (color 0 0 0 0))
@@
   )
   (wire (pts (xy 177.8 57.15) (xy 234.315 57.15))
-    (stroke (width 0) (type default) (color 0 0 0 0))
-  )
-  (wire (pts (xy 184.15 144.145) (xy 196.85 144.145))
     (stroke (width 0) (type default) (color 0 0 0 0))
   )
@@
     (pin "1")
   )
-  (symbol (lib_id "power:+5V") (at 182.88 29.845 0)
-    (in_bom yes) (on_board yes) (fields_autoplaced)
-    (property "Reference" "#PWR043" (id 0) (at 182.88 33.655 0)
-      (effects (font (size 1.27 1.27)) hide)
-    )
-    (property "Value" "+5V" (id 1) (at 182.88 26.2405 0))
-    (property "Footprint" "" (id 2) (at 182.88 29.845 0)
-      (effects (font (size 1.27 1.27)) hide)
-    )
-    (property "Datasheet" "" (id 3) (at 182.88 29.845 0)
+  (symbol (lib_id "power:+5V") (at 224.155 29.845 0)
+    (in_bom yes) (on_board yes) (fields_autoplaced)
+    (property "Reference" "#PWR043" (id 0) (at 224.155 33.655 0)
+      (effects (font (size 1.27 1.27)) hide)
+    )
+    (property "Value" "+5V" (id 1) (at 224.155 26.2405 0))
+    (property "Footprint" "" (id 2) (at 224.155 29.845 0)
+      (effects (font (size 1.27 1.27)) hide)
+    )
+    (property "Datasheet" "" (id 3) (at 224.155 29.845 0)
       (effects (font (size 1.27 1.27)) hide)
     )
@@
       (effects (font (size 1.27 1.27)) hide)
     )
-    (pin "1")
-    (pin "2")
-    (pin "3")
+    (pin "10")
+    (pin "8")
+    (pin "9")
   )
   (symbol (lib_id "Device:R") (at 248.285 38.1 0)
@@
     (pin "1")
     (pin "2")
+  )
+  (symbol (lib_id "power:GND") (at 210.82 117.475 0)
+    (in_bom yes) (on_board yes) (fields_autoplaced)
+    (property "Reference" "#PWR?" (id 0) (at 210.82 123.825 0)
+      (effects (font (size 1.27 1.27)) hide)
+    )
+    (property "Value" "GND" (id 1) (at 210.82 122.0375 0))
+    (property "Footprint" "" (id 2) (at 210.82 117.475 0)
+      (effects (font (size 1.27 1.27)) hide)
+    )
+    (property "Datasheet" "" (id 3) (at 210.82 117.475 0)
+      (effects (font (size 1.27 1.27)) hide)
+    )
+    (pin "1")
   )
   (symbol (lib_id "Device:R") (at 227.33 38.1 0)
@@
       (effects (font (size 1.27 1.27)) hide)
     )
-    (pin "1")
-    (pin "2")
-    (pin "3")
+    (pin "11")
+    (pin "12")
+    (pin "13")
   )
   (symbol (lib_id "Device:R") (at 199.39 38.1 0)
@@
     )
     (property "Datasheet" "~" (id 3) (at 234.315 38.1 0)
-      (effects (font (size 1.27 1.27)) hide)
-    )
-    (pin "1")
-    (pin "2")
-  )
-  (symbol (lib_id "Device:C") (at 184.15 147.955 0)
-    (in_bom yes) (on_board yes) (fields_autoplaced)
-    (property "Reference" "C7" (id 0) (at 187.071 147.0465 0)
-      (effects (font (size 1.27 1.27)) (justify left))
-    )
-    (property "Value" "100nF" (id 1) (at 187.071 149.8216 0)
-      (effects (font (size 1.27 1.27)) (justify left))
-    )
-    (property "Footprint" "Capacitor_THT:C_Disc_D3.8mm_W2.6mm_P2.50mm" (id 2) (at 185.1152 151.765 0)
-      (effects (font (size 1.27 1.27)) hide)
-    )
-    (property "Datasheet" "~" (id 3) (at 184.15 147.955 0)
       (effects (font (size 1.27 1.27)) hide)
     )
@@
     (pin "3")
   )
+  (symbol (lib_id "power:GND") (at 156.845 35.56 0) (mirror y)
+    (in_bom yes) (on_board yes) (fields_autoplaced)
+    (property "Reference" "#PWR0104" (id 0) (at 156.845 41.91 0)
+      (effects (font (size 1.27 1.27)) hide)
+    )
+    (property "Value" "GND" (id 1) (at 156.845 40.1225 0))
+    (property "Footprint" "" (id 2) (at 156.845 35.56 0)
+      (effects (font (size 1.27 1.27)) hide)
+    )
+    (property "Datasheet" "" (id 3) (at 156.845 35.56 0)
+      (effects (font (size 1.27 1.27)) hide)
+    )
+    (pin "1")
+  )
   (symbol (lib_id "74xx:74LS51") (at 89.535 84.455 180)
     (in_bom yes) (on_board yes)
@@
       (effects (font (size 1.27 1.27)) hide)
     )
-    (pin "1")
-    (pin "10")
-    (pin "11")
-    (pin "12")
-    (pin "13")
-    (pin "8")
-    (pin "9")
+    (pin "2")
+    (pin "3")
+    (pin "4")
+    (pin "5")
+    (pin "6")
   )
   (symbol (lib_id "74xx:74LS51") (at 212.725 147.955 0)
@@
       (effects (font (size 1.27 1.27)) hide)
     )
-    (pin "1")
-    (pin "10")
-    (pin "11")
-    (pin "12")
-    (pin "13")
-    (pin "8")
-    (pin "9")
+    (pin "14")
+    (pin "7")
   )
   (symbol (lib_id "74xx:74LS00") (at 93.345 40.005 0) (mirror y)
@@
       (effects (font (size 1.27 1.27)) hide)
     )
-    (pin "1")
-    (pin "2")
-    (pin "3")
+    (pin "4")
+    (pin "5")
+    (pin "6")
   )
   (symbol (lib_id "74xx:74LS00") (at 233.045 147.955 0)
@@
       (effects (font (size 1.27 1.27)) hide)
     )
-    (pin "1")
-    (pin "2")
-    (pin "3")
+    (pin "14")
+    (pin "7")
   )
   (symbol (lib_id "power:+5V") (at 212.725 135.255 0)
@@
       (effects (font (size 1.27 1.27)) hide)
     )
-    (pin "1")
-  )
-  (symbol (lib_id "power:+5V") (at 210.82 109.855 0)
-    (in_bom yes) (on_board yes) (fields_autoplaced)
-    (property "Reference" "#PWR044" (id 0) (at 210.82 113.665 0)
-      (effects (font (size 1.27 1.27)) hide)
-    )
-    (property "Value" "+5V" (id 1) (at 210.82 106.2505 0))
-    (property "Footprint" "" (id 2) (at 210.82 109.855 0)
-      (effects (font (size 1.27 1.27)) hide)
-    )
-    (property "Datasheet" "" (id 3) (at 210.82 109.855 0)
-      (effects (font (size 1.27 1.27)) hide)
-    )
