File: intellivision t-card replic/intellivision t-card replic.kicad_sch (KiCad schematic)
At the start: 6 parts, among them J1 2x22 card edge connector, U1 74LS374, U2 74LS374, U3 74LS42, U4 74LS04, U5 74LS08

Commit message: partial layout
Parts:
- added C1, C3, C5, C7, C9: 100nF, Capacitor_THT:C_Disc_D3.8mm_W2.6mm_P2.50mm, symbol Device:C
Connections:
- net +5V: now also C1.1, C3.1, C5.1, C7.1, C9.1
- net GND: now also C1.2, C3.2, C5.2, C7.2, C9.2
