File: intellivision t-card replic/intellivision t-card replic.kicad_pcb (KiCad board)
At the start: 2 copper layers, 58.2 x 8.8 mm, 70 parts, among them J1 2x22 card edge connector, SW1 SW_DIP_x08, SW2 SW_DIP_x08, SW3 SW_DIP_x08, SW4 SW_DIP_x08, U1 74LS374, U10 74LS00, U11 74LS85, U12 74LS51, U13 74LS00, U14 74LS85, U15 74LS51, U16 74LS00, U17 74LS85, U18 2732, U19 2732, U2 74LS374, U20 2732, U21 2732, U22 2732, U23 2732, U24 2732, U25 2732, U3 74LS42, U4 74LS04, U5 74LS08, U6 74LS51, U7 74LS00, U8 74LS85, U9 74LS51

Commit message: some layout started
Parts:
- moved U22 446.6 mm to (208.3, 91.4), turned to 90 degrees
- moved U18 431.5 mm to (208.3, 114.3), turned to 90 degrees
- moved U19 426.9 mm to (142.2, -156.2), turned to 90 degrees
- moved R1 423.3 mm to (285.0, 95.8)
- moved R5 423.3 mm to (271.7, 95.8)
- moved R7 423.3 mm to (258.4, 96.6)
- moved R8 423.3 mm to (280.6, 91.7)
- moved SW1 423.3 mm to (258.7, 73.5)
- moved U7 423.3 mm to (280.7, 72.4)
- moved R2 423.3 mm to (302.3, 76.4)
- moved R3 423.3 mm to (293.9, 91.7)
- moved R4 423.3 mm to (302.3, 80.4)
- moved R6 423.3 mm to (302.3, 72.3)
- moved U6 423.3 mm to (291.5, 72.4)
- moved U8 423.3 mm to (269.8, 72.4)
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Other:
- board size 58.2 x 8.8 mm -> 143 x 165.9 mm
- board text added: "1"
- board text added: "2"
- board text added: "3"
- board text added: "4"

Commit message: partial layout
Parts:
- added C10: 100nF, Capacitor_THT:C_Disc_D3.8mm_W2.6mm_P2.50mm, F.Cu at (180.4, 89.5)
- added C11: 100nF, Capacitor_THT:C_Disc_D3.8mm_W2.6mm_P2.50mm, F.Cu at (153.7, 89.5)
- added C12: 100nF, Capacitor_THT:C_Disc_D3.8mm_W2.6mm_P2.50mm, F.Cu at (86.0, 89.5)
- added C13: 100nF, Capacitor_THT:C_Disc_D3.8mm_W2.6mm_P2.50mm, F.Cu at (56.5, 111.8)
- added C9: 100nF, Capacitor_THT:C_Disc_D3.8mm_W2.6mm_P2.50mm, F.Cu at (114.3, 121.9)
- moved R14 317.5 mm to (121.3, 66.7)
- moved R12 301.8 mm to (146.7, 66.7), turned to 180 degrees
- moved SW2 286.8 mm to (139.1, 52.7), turned to -90 degrees
- moved R9 286.4 mm to (150.5, 47.6), turned to -90 degrees
- moved R11 286.2 mm to (146.7, 64.1), turned to 180 degrees
- moved R13 283.2 mm to (121.3, 64.1)
- moved C8 282.2 mm to (64.8, 45.7), turned to 180 degrees
- moved C6 281.8 mm to (106.0, 45.7), turned to 180 degrees
- moved U9 281.2 mm to (150.5, 41.3), turned to 180 degrees
- moved U10 281.2 mm to (139.7, 41.3), turned to 180 degrees
- moved U11 281.2 mm to (128.9, 41.3), turned to 180 degrees
- moved R22 279.4 mm to (87.6, 66.7)
- moved SW3 275.4 mm to (105.4, 52.7), turned to -90 degrees
- moved R20 274.2 mm to (113.0, 66.7), turned to 180 degrees
- moved R15 267.2 mm to (145.4, 47.6), turned to -90 degrees
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- renumbered R9 to R10, R16 to R15, R15 to R16, R18 to R17, R17 to R18, R24 to R23, R23 to R24, R26 to R25, R25 to R26, R32 to R31, R31 to R32, R8 to R7, R7 to R8, R10 to R9
Connections:
- R10 pad 2: Net-(R9-Pad2) -> /Rom Section Intellivision 2/ena
- R15 pad 2: Net-(R16-Pad2) -> Net-(R15-Pad2)
- R16 pad 2: Net-(R15-Pad2) -> Net-(R16-Pad2)
- R17 pad 2: /Rom Section Intellivision 3/ena -> Net-(R17-Pad2)
- R18 pad 2: Net-(R17-Pad2) -> /Rom Section Intellivision 3/ena
- R23 pad 2: Net-(R24-Pad2) -> Net-(R23-Pad2)
- R24 pad 2: Net-(R23-Pad2) -> Net-(R24-Pad2)
- R25 pad 2: /Rom Section Intellivision 4/ena -> Net-(R25-Pad2)
- R26 pad 2: Net-(R25-Pad2) -> /Rom Section Intellivision 4/ena
- R31 pad 2: Net-(R32-Pad2) -> Net-(R31-Pad2)
- R32 pad 2: Net-(R31-Pad2) -> Net-(R32-Pad2)
- R7 pad 2: Net-(R8-Pad2) -> Net-(R7-Pad2)
- R8 pad 2: Net-(R7-Pad2) -> Net-(R8-Pad2)
- R9 pad 2: /Rom Section Intellivision 2/ena -> Net-(R9-Pad2)
- SW1 pad 10: +5V -> GND
- SW1 pad 11: +5V -> GND
- SW1 pad 12: +5V -> GND
- SW1 pad 13: +5V -> GND
- SW1 pad 14: +5V -> GND
- SW1 pad 15: +5V -> GND
- SW1 pad 16: unconnected-(SW1-Pad16) -> GND
- SW1 pad 9: +5V -> GND
- SW2 pad 10: +5V -> GND
- SW2 pad 11: +5V -> GND
- SW2 pad 12: +5V -> GND
- SW2 pad 13: +5V -> GND
- SW2 pad 14: +5V -> GND
- SW2 pad 15: +5V -> GND
- SW2 pad 16: unconnected-(SW2-Pad16) -> GND
- SW2 pad 9: +5V -> GND
- SW3 pad 10: +5V -> GND
- SW3 pad 11: +5V -> GND
- SW3 pad 12: +5V -> GND
- SW3 pad 13: +5V -> GND
- SW3 pad 14: +5V -> GND
- SW3 pad 15: +5V -> GND
- SW3 pad 16: unconnected-(SW3-Pad16) -> GND
- SW3 pad 9: +5V -> GND
- SW4 pad 10: +5V -> GND
- SW4 pad 11: +5V -> GND
- SW4 pad 12: +5V -> GND
- SW4 pad 13: +5V -> GND
- SW4 pad 14: +5V -> GND
- SW4 pad 15: +5V -> GND
- SW4 pad 16: unconnected-(SW4-Pad16) -> GND
- SW4 pad 9: +5V -> GND
- U10 pad 1: +5V -> GND
- U10 pad 2: +5V -> GND
- U13 pad 1: +5V -> GND
- U13 pad 2: +5V -> GND
- U16 pad 1: +5V -> GND
- U16 pad 2: +5V -> GND
- U7 pad 1: +5V -> GND
- U7 pad 2: +5V -> GND
Routing:
- net GND: track 0.00 -> 1431.7 mm, vias 0 -> 6
- net +5V: track 0.00 -> 824.3 mm, vias 0 -> 1
- net a3: track 0.00 -> 286.5 mm, vias 0 -> 3
- net a2: track 0.00 -> 272.8 mm, vias 0 -> 3
- net /intellivision roms/DWS or BAR: track 0.00 -> 269.6 mm, vias 0 -> 3
- net a7: track 0.00 -> 267.7 mm, vias 0 -> 3
- net a1: track 0.00 -> 264.2 mm
- net /Rom Section Intellivision 1/DW: track 0.00 -> 253.1 mm
- net a0: track 0.00 -> 252.9 mm, vias 0 -> 2
- net a6: track 0.00 -> 216.1 mm, vias 0 -> 3
- net a5: track 0.00 -> 212.0 mm, vias 0 -> 3
- net a4: track 0.00 -> 209.2 mm, vias 0 -> 3
- net a8: track 0.00 -> 198.5 mm, vias 0 -> 3
- net a9: track 0.00 -> 198.3 mm, vias 0 -> 3
- net d7: track 0.00 -> 165.8 mm, vias 0 -> 3
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Other:
- board text removed: "1"
- board text removed: "2"
- board text removed: "3"
- board text removed: "4"

Commit message: layout 'finished', needs cleanup
Routing:
- net a12: track 103.8 -> 347.1 mm
- net a13: track 104.2 -> 325.0 mm
- net a14: track 103.9 -> 319.0 mm
- net a11: track 159.2 -> 366.6 mm
- net a15: track 104.1 -> 306.6 mm
- net /Rom Section Intellivision 2/oa (bank) inverted at 74ls04: track 26.2 -> 225.8 mm, vias 1 -> 3
- net d15: track 120.5 -> 258.5 mm, vias 3 -> 4
- net d3: track 121.3 -> 257.2 mm, vias 0 -> 1
- net d12: track 107.5 -> 242.3 mm, vias 3 -> 4
- net d11: track 111.0 -> 244.1 mm, vias 2 -> 3
- net d13: track 111.8 -> 244.3 mm, vias 3 -> 4
- net d14: track 116.1 -> 243.0 mm, vias 3 -> 4
- net d7: track 165.8 -> 291.3 mm, vias 3 -> 4
- net a10: track 164.7 -> 286.5 mm, vias 0 -> 2
- net d6: track 160.8 -> 281.6 mm, vias 3 -> 4
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
Commit message: layout probably done (minus silk and copper text)
Routing:
- net d9: track 204.2 -> 211.5 mm
- net a9: track 271.0 -> 277.8 mm
- net a10: track 286.5 -> 279.7 mm, vias 2 -> 0
- net GND: track 1494.9 -> 1500.6 mm
- net bc1: track 38.8 -> 33.8 mm
- net /Rom Section Intellivision 1/oa (bank) inverted at 74ls04: track 168.6 -> 164.1 mm
- net bc2: track 33.7 -> 30.2 mm
- net /intellivision roms/a11_1: track 100.7 -> 97.3 mm
- net d7: track 291.3 -> 288.1 mm
- net /intellivision roms/a11_4: track 123.9 -> 120.7 mm
- net d15: track 258.5 -> 255.4 mm
- net bdir: track 29.1 -> 26.3 mm
- net d0: track 231.7 -> 229.1 mm
- net a8: track 266.9 -> 269.5 mm
- net d13: track 244.3 -> 242.5 mm
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- added copper zone on B.Cu, net +5V
- added copper zone on F.Cu, net GND

Commit message: layout cleanup
Parts:
- added G***: LOGO, Evan's misc parts:Evan Logo, B.Cu at (50.2, 21.0)
- added G***: LOGO, Evan's misc parts:OSHW gear, B.Cu at (184.2, 21.6)
Routing:
- net /Rom Section Intellivision 1/DW: track 347.1 -> 342.6 mm
- net Net-(R21-Pad2): track 52.1 -> 48.9 mm
- net Net-(R13-Pad2): track 52.2 -> 49.6 mm
- net /Rom Section Intellivision 4/oa (bank) inverted at 74ls04: track 156.1 -> 153.5 mm
- net Net-(U10-Pad8): track 37.9 -> 40.4 mm
- net Net-(R5-Pad2): track 52.6 -> 50.1 mm
- net /Rom Section Intellivision 4/ena: track 36.8 -> 38.7 mm
- net Net-(U15-Pad13): track 41.7 -> 43.7 mm
- net Net-(R14-Pad2): track 49.5 -> 47.7 mm
- net Net-(U15-Pad3): track 51.0 -> 52.7 mm
- net Net-(R22-Pad2): track 49.5 -> 47.8 mm
- net Net-(R6-Pad2): track 50.1 -> 48.7 mm
- net /Rom Section Intellivision 2/oa (bank) inverted at 74ls04: track 227.0 -> 225.8 mm
- net a3: track 286.5 -> 287.7 mm
- net a11: track 366.6 -> 365.4 mm
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Other:
- board text added: "5859-3229-PR"
- board text added: "A12"
- board text added: "A13"
- board text added: "A14"
- board text added: "A15"
- board text added: "Circuit Lab"
- board text added: "ENA"
- board text added: "Intellivision T-card for use with RAM or standard parallel ROMs"
- board text added: "MATTEL INC. © 1982 T-CARD ASSY 5859-9229-PR"
- board text added: "NC"
- board text added: "RAM"
- board text added: "RAMH"
- board text added: "T-CARD"
- board text added: "abzman2k.wordpress.com"
